File: esp32_cnc_shield.kicad_pcb (KiCad board)
At the start: 2 copper layers, 101.6 x 64.8 mm, 18 parts, among them J1 USB C, J10 Z Engine, J2 UART, J3 X Mode, J4 External Power, J5 X Engine, J6 Y Mode, J7 Configuration, J8 Y Engine, J9 Z Mode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

Commit message: Make it pretty
Parts:
- added G***: LOGO, pretty:alpaca-pica, F.Cu at (154.9, 113.0)

Commit message: Add pseudo shottky
Parts:
- added J11: Future Shottky, Connector_PinHeader_2.54mm:PinHeader_1x02_P2.54mm_Vertical, F.Cu at (163.8, 103.5)
- moved G*** 3.18 mm to (158.1, 113.0)
Connections:
- net USB_PWR renamed VCC
- U1 pad 18: unconnected-(U1-Pad18) -> VIN
Routing:
- net VIN: track 0.00 -> 39.7 mm
- net VCC: track 155.0 -> 162.9 mm
